File: portiqo-key-hw/pcb/portiqo-key.kicad_sch (KiCad schematic)
At the start: 129 parts, among them IC1 GS358-FR, J1 JRG01-002, J2 JRG01-002, J3 JRG01-002, J4 JRG01-002, Q1 WNM3013-3/TR, Q2 WNM3013-3/TR, Q3 WNM3013-3/TR, Q4 CJE3139K, U2 nRF52840, U3 BL8064CB3TR33, U4 LGS4056HDA-420, U5 Ci522, X1 32MHZ X201632MOB4SI, X2 32.768KHz, X3 27.12MHZ X2016712MMB4SI

Commit message: Updated schematic for wireless charging. Added footprints for most ICs
Parts:
- removed C49: 1uF, symbol Device:C
- removed IC1: GS358-FR, Package_SO:VSSOP-8_3x3mm_P0.65mm, symbol Amplifier_Operational:OPA2196xDGK
- removed JP1: Conn_01x02, Connector_PinHeader_1.00mm:PinHeader_1x02_P1.00mm_Vertical, symbol Connector_Generic:Conn_01x02
- removed KEY1, KEY2: SW_SPST, symbol Switch:SW_SPST
- removed LED1, LED2, LED3, LED4, LED5, LED6, LED7, LED8: MHPA0606RGBDT, symbol Device:LED_RGBA
- removed LED10, LED9: LED, symbol Device:LED
- removed R22, R23: 5.1K, symbol Device:R
- removed R26: 20K, symbol Device:R
- removed R28: 2K, symbol Device:R
- removed U4: LGS4056HDA-420, symbol Battery_Management:LGS4056HDA-420
- removed USB1: USB_C_Receptacle_USB2.0_14P, symbol Connector:USB_C_Receptacle_USB2.0_14P
- added C23, C39, C51: 100nF, Capacitor_SMD:C_0402_1005Metric, symbol Device:C
- added C50: 1uF, Capacitor_SMD:C_0402_1005Metric, symbol Device:C
- added C59: 2.2uF, Capacitor_SMD:C_0402_1005Metric, symbol Device:C
- added C60, C61: 10uF, Capacitor_SMD:C_0402_1005Metric, symbol Device:C
- added C62: .183uF, Capacitor_SMD:C_0402_1005Metric, symbol Device:C
- added C63: 1900pF, Capacitor_SMD:C_0402_1005Metric, symbol Device:C
- added C64, C65: .47uF 25v, Capacitor_SMD:C_0402_1005Metric, symbol Device:C
- added C66, C67: 22nF 25v, Capacitor_SMD:C_0402_1005Metric, symbol Device:C
- added C68: 10nF 10v, Capacitor_SMD:C_0402_1005Metric, symbol Device:C
- added C69: 10nf 10v, Capacitor_SMD:C_0402_1005Metric, symbol Device:C
- added J6: Qi Coil, symbol Connector_Generic:Conn_01x02
- added JP2: BATTERY, symbol Connector_Generic:Conn_01x02
- added R29: 196, Resistor_SMD:R_0402_1005Metric, symbol Device:R
- added R30: 20k, Resistor_SMD:R_0402_1005Metric, symbol Device:R
- added R31: 10K, Resistor_SMD:R_0402_1005Metric, symbol Device:R
- added R32: .82, Resistor_SMD:R_0402_1005Metric, symbol Device:R
- added R33: 2.21K, Resistor_SMD:R_0402_1005Metric, symbol Device:R
- added R34: 221, Resistor_SMD:R_0402_1005Metric, symbol Device:R
- added U4: GS358-FR, Package_DFN_QFN:DFN-8-1EP_2x2mm_P0.5mm_EP0.9x1.3mm, symbol Amplifier_Operational:GS358
- added U6: BQ29707, Package_SON:WSON-6_1.5x1.5mm_P0.5mm, symbol Battery_Management:BQ297xy
- added U7: BQ25100YFPR, BQ25100:YFP0006AFAV, symbol BQ25100:BQ25100YFPR
- added U8: BQ51003YFPR, BQ51003:YFP0028APAL, symbol BQ51003:BQ51003YFPR
- added U9: CSD85301Q2, CSD85301Q2:DQK0006B, symbol CSD85301Q2:CSD85301Q2
- C1, C10, C11, C12, C13, C14, C15, C16, C17, C18, C2, C20, C21, C22, C24, C25, C26, C27, C28, C29, C3, C31, C33, C34, C35, C36, C37, C38, C4, C40, C41, C42, C43, C44, C45, C46, C47, C5, C6, C7, C8, C9: footprint (none) -> Capacitor_SMD:C_0402_1005Metric
- C19, C30, C32: value 100nf -> 100nF; footprint (none) -> Capacitor_SMD:C_0402_1005Metric
- C48: value 4.7uf -> 4.7uF; footprint (none) -> Capacitor_SMD:C_0402_1005Metric
- L1, L5, L6: footprint (none) -> Inductor_SMD:L_0402_1005Metric
- L2, L3, L4: footprint (none) -> Inductor_SMD:L_0603_1608Metric
- Q1, Q2: footprint (none) -> Package_TO_SOT_SMD:SOT-723
- Q3: footprint (none) -> Package_TO_SOT_SMD:SOT-723; LCSC Link (none) -> https://lcsc.com/product-detail/MOSFETs_WILLSEMI-Will-Semic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
- Q4: footprint (none) -> Package_TO_SOT_SMD:SOT-523
- R1, R10, R11, R12, R13, R14, R15, R16, R17, R18, R2, R25, R27, R3, R4, R5, R6, R7, R8, R9: footprint (none) -> Resistor_SMD:R_0402_1005Metric
- R19, R21: value 1K -> 10K; footprint (none) -> Resistor_SMD:R_0402_1005Metric
- R20: value 1K -> 13K; footprint (none) -> Resistor_SMD:R_0402_1005Metric
- R24: value 2K -> 4.7K; footprint (none) -> Resistor_SMD:R_0402_1005Metric
- TP1, TP10, TP11, TP12, TP13, TP2, TP3, TP4, TP5, TP6, TP7, TP8: footprint (none) -> TestPoint:TestPoint_Pad_D1.0mm
- TP9: renamed from TP1; footprint (none) -> TestPoint:TestPoint_Pad_D1.0mm
- U1: value ~ -> RS2257XC6; footprint (none) -> Package_TO_SOT_SMD:SOT-363_SC-70-6
- U5: footprint (none) -> Package_DFN_QFN:QFN-16-1EP_3x3mm_P0.5mm_EP1.9x1.9mm
- X1, X3: footprint (none) -> Crystal:Crystal_SMD_2016-4Pin_2.0x1.6mm
- X2: footprint (none) -> Crystal:SMD1610-2P X161032768KGD2SI CRYSTAL
Connections:
- net BAT: now also C50.1, JP2.1 (Pin_1), R34.1, U7.A1 (OUT)
- net GND: now also R19.2, R20.2, R21.2, C23.2, C39.2, C50.2, C59.2, C60.2, C61.2, R29.2, R31.2, R32.2, R33.2, U7.C2 (VSS), U8.A1 (PGND), U8.A2 (PGND), U8.A3 (PGND), U8.A4 (PGND), U8.G2 (EN2), U8.G3 (EN1), U8.G4 (AD)
- net LED_B_H: no longer R21.1, U2.AD22 (TRACEDATA0/P1.00)
- net LF_AMP_PWR: now also U4.8 (VDD)
- net LF_Env_Dete: now also U4.2 (-)
- net LF_O1A: now also U4.1
- net LF_OA_OUT: now also U4.7
- net LF_VBIAS: now also U4.3 (+), U4.5 (+)
- net VCC3.3V: now also C39.1; no longer R24.1
- net at C37.1, R15.2: now also U4.6 (-)
- net at R24.2: now also R29.1, R30.2, U8.F2 (FOD)
- net KEY_A: no longer names the net of U2.G1 (P0.26)
- net KEY_B: no longer names the net of U2.W24 (P1.02)
- net LED1: no longer names the net of U2.L1 (P0.06)
- net LED2: no longer names the net of U2.N1 (P0.08)
- net LED3: no longer names the net of U2.R1 (TRACEDATA3/P1.09)
- net LED4: no longer names the net of U2.U1 (TRACEDATA1/P0.12)
- net LED5: no longer names the net of U2.AD8 (P0.13)
- net LED6: no longer names the net of U2.AD10 (P0.15)
- net LED7: no longer names the net of U2.AD12 (P0.17)
- net LED8: no longer names the net of U2.AD16 (P0.20)
- net LED_FIELD: no longer names the net of U2.Y23 (P1.01)
- net LED_G_H: no longer names the net of R20.1
- net LED_G_H: now also U7.B2 (ISET); no longer U2.AD18 (P0.22)
- net LED_R_H: no longer names the net of U2.AD20 (P0.24)
- net LED_R_H: no longer R19.1
- net VUSB renamed VQI
- net VQI: now also C23.1, C59.1, U7.A2 (IN), U8.D1 (OUT), U8.D2 (OUT), U8.D3 (OUT), U8.D4 (OUT)
- new net: C63.2, C65.1, C67.1, C69.1, J6.1 (Pin_1), U8.B1 (AC2), U8.B2 (AC2)
- new net: C62.2, C63.1, C64.1, C66.1, C68.1, U8.B3 (AC1), U8.B4 (AC1)
- new net: C69.2, U8.C1 (BOOT2)
- new net: C68.2, U8.C4 (BOOT1)
- new net: C67.2, U8.E1 (COMM2)
- new net: C65.2, U8.E2 (CLAMP2)
- new net: C64.2, U8.E3 (CLAMP1)
- new net: C66.2, U8.E4 (COMM1)
- new net: R31.1, U8.F1 (TS-CTRL)
- new net: R24.1, U8.G1 (ILIM)
- new net: C62.1, J6.2 (Pin_2)
- new net: C51.1, R34.2, U6.5 (BAT)
- new net: C51.2, JP2.2 (Pin_2), U6.4 (VSS), U9.4 (S2)
- new net: U9.3 (D2), U9.6 (D1)
- new net: U6.3 (Dout), U9.5 (G2)
- new net: U9.7 (D1), U9.8 (D2)
- new net: R33.1, U6.6 (V-)
- new net: R32.1, U9.1 (S1)
- new net: U6.2 (Cout), U9.2 (G1)
- new net: R21.1, U7.B1 (TS)
- new net: R19.1, U7.C1 (PRETERM)
- new net AD-EN: U8.F3 (AD-EN_N)
- new net CHG: U8.F4 (CHG_N)
- new net RECT: C60.1, C61.1, R30.1, U8.C2 (RECT), U8.C3 (RECT)
- no-connect marks 26 -> 38
Other:
- moved on the sheet: C25, C26, C27, C30, C9

Commit message: HW V0.1
Parts:
- removed J1, J2, J3, J4: JRG01-002, symbol Connector_Generic:Conn_01x01
- removed TP1, TP10, TP11, TP12, TP13, TP2, TP3, TP4, TP5, TP6, TP7, TP8, TP9: TestPoint, TestPoint:TestPoint_Pad_D1.0mm, symbol Connector:TestPoint
- added J1, J2: Conn_02x03_Counter_Clockwise, Connector:Tag-Connect_TC2030-IDC-NL_2x03_P1.27mm_Vertical, symbol Connector_Generic:Conn_02x03_Counter_Clockwise
- added L7: 2.7nH, Inductor_SMD:L_0402_1005Metric, symbol Device:L
- A1: value CA-C01 -> 2450AT18A100; footprint (none) -> RF_Antenna:Johanson_2450AT18x100
- C21: value 0.8pF -> 1pF
- J6, JP2: footprint (none) -> Jumper:Solderpad - 2 pin
- U8: value BQ51003YFPR -> BQ51013B; footprint BQ51003:YFP0028APAL -> BQ51013B:RHL20_2P05X3P05
- X3: Substitute (none) -> SX1B27.120F1210F30
Connections:
- net LF_Evn_Dete is gone; now on net LF_Env_Dete: C36.1, R9.2
- net LF_O1A is gone; now on net LF_OA1: C38.2, R17.2, U4.1
- net P_LF_ANT_RAW is gone; now on net LF-ANT: C10.1, C33.1, C34.1, VD1.2 (A)
- net AD-EN: now also U8.8 (AD-EN_N); no longer U8.F3 (AD-EN_N)
- net BAT: now also J1.6 (Pin_6)
- net BLE_ANT: now also C21.2; no longer C21.1, L5.2
- net CHG: now also U8.7 (CHG_N); no longer U8.F4 (CHG_N)
- net GND: now also U4.4 (VSS), U8.1 (PGND), U8.10 (EN1), U8.11 (EN2), U8.20 (PGND), U8.9 (AD), J1.2 (Pin_2), L7.2; no longer A1.1, A1.2, C21.2, L5.1, U8.A1 (PGND), U8.A2 (PGND), U8.A3 (PGND), U8.A4 (PGND), U8.G2 (EN2), U8.G3 (EN1), U8.G4 (AD)
- net LF_AMP_PWR: now also J2.4 (Pin_4)
- net LF_ANT_DRV: now also J2.2 (Pin_2)
- net LF_MOD: now also J2.1 (Pin_1)
- net LF_OA_OUT: now also J2.3 (Pin_3)
- net LF_RSSI: now also J2.5 (Pin_5)
- net NFC_ANT_SEL: now also J2.6 (Pin_6)
- net RECT: now also U8.18 (RECT); no longer U8.C2 (RECT), U8.C3 (RECT)
- net SWCLK: now also J1.5 (Pin_5)
- net VCC3.3V: now also J1.4 (Pin_4)
- net VQI: now also U8.4 (OUT); no longer U8.D1 (OUT), U8.D2 (OUT), U8.D3 (OUT), U8.D4 (OUT)
- net at C63.2, C65.1, C67.1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: now also U8.19 (AC2); no longer U8.B1 (AC2), U8.B2 (AC2)
- net at C62.2, C63.1, C64.1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: now also U8.2 (AC1); no longer U8.B3 (AC1), U8.B4 (AC1)
- net at C69.2: now also U8.17 (BOOT2); no longer U8.C1 (BOOT2)
- net at C68.2: now also U8.3 (BOOT1); no longer U8.C4 (BOOT1)
- net at C67.2: now also U8.15 (COMM2); no longer U8.E1 (COMM2)
- net at C65.2: now also U8.16 (CLAMP2); no longer U8.E2 (CLAMP2)
- net at C64.2: now also U8.5 (CLAMP1); no longer U8.E3 (CLAMP1)
- net at C66.2: now also U8.6 (COMM1); no longer U8.E4 (COMM1)
- net at R31.1: now also U8.13 (TS-CTRL); no longer U8.F1 (TS-CTRL)
- net at R24.2, R29.1, R30.2: now also U8.14 (FOD); no longer U8.F2 (FOD)
- net at R24.1: now also U8.12 (ILIM); no longer U8.G1 (ILIM)
- net RESET: now reaches U2.AC13 (P0.18/~{RESET})
- net RESET: now also J1.1 (Pin_1)
- net P_LF_ANT_DRV renamed LF-ANT
- new net: C21.1, L5.2, L7.1
- new net: A1.2, L5.1
- new net SWIO: J1.3 (Pin_3)
- no-connect marks 38 -> 37
Other:
- moved on the sheet: A1, C1, C11, C12, C13, C14, C15, C16, C17, C18, C19, C2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
